File: src/kicad/Timer.kicad_pcb (KiCad board)
At the start: 2 copper layers, 84.5 x 100.8 mm, 47 parts, among them J1 Conn_01x02, Q2 Q_NPN_BCE, SW10 SW_DIP_x01, SW3 SW_SP4T_NR01104, SW4 SW_DIP_x01, SW5 SW_DIP_x01, SW6 SW_DIP_x01, SW7 SW_DIP_x01, SW8 SW_DIP_x01, SW9 SW_DIP_x01, U1 4060, U2 NE555P, U3 NE555P

Commit message: Add files via upload
Parts:
- U1: footprint Package_SO:SOIC-16W_5.3x10.2mm_P1.27mm -> Package_DIP:DIP-16_W7.62mm
- moved U1 14.3 mm to (126.8, 92.5)
- renumbered 1 to D1, 2 to D2, 4 to D3, 8 to D4, 16 to D5, 32 to D6, 64 to D7, Dismiss to SW2
Routing:
- net GND: track 108.4 -> 0.00 mm
- net Net-(D7-A): track 19.3 -> 10.3 mm
- net VCC: track 33.4 -> 24.5 mm
- net Net-(D4-A): track 37.6 -> 30.9 mm
- net Net-(Q2-E): track 171.7 -> 165.0 mm
- net Net-(D3-A): track 20.2 -> 14.1 mm
- net Net-(D5-A): track 10.7 -> 5.34 mm
- net Net-(U1-CLR): track 102.4 -> 97.3 mm
- net Net-(D2-A): track 11.6 -> 8.10 mm
- net Net-(D6-A): track 6.07 -> 8.42 mm
- net Net-(U1-~{Φ1}): track 7.99 -> 10.1 mm
- net Net-(U1-Φ0): track 13.2 -> 14.7 mm
- net Net-(U1-~{Φ0}): track 14.7 -> 15.6 mm

Commit message: Add files via upload
Parts:
- removed SW10: SW_DIP_x01, Button_Switch_THT:SW_PUSH_6mm
- added SW1: SW_Push, Button_Switch_THT:SW_PUSH_6mm, F.Cu at (101.2, 109.2)
- SW4, SW5, SW6, SW7, SW8, SW9: value SW_DIP_x01 -> SW_Push
- moved SW7 65.3 mm to (164.2, 97.2)
- moved SW8 22.1 mm to (164.2, 108.2), turned to 180 degrees
- moved SW4 16.8 mm to (94.8, 93.8), turned to 0 degrees
- moved SW6 16.3 mm to (94.8, 73.8), turned to 0 degrees
- moved SW9 12.7 mm to (164.2, 86.2), turned to 180 degrees
- moved SW5 10.3 mm to (101.2, 88.2)
Connections:
- SW4 pad 1: Net-(R3-Pad2) -> Net-(R5-Pad2)
- SW5 pad 1: Net-(R5-Pad2) -> Net-(R6-Pad2)
- SW6 pad 1: Net-(R6-Pad2) -> Net-(R7-Pad2)
- SW7 pad 1: Net-(R7-Pad2) -> Net-(R8-Pad2)
- SW8 pad 1: Net-(R10-Pad2) -> Net-(R9-Pad2)
- SW9 pad 1: Net-(R8-Pad2) -> Net-(R10-Pad2)
Routing:
- net unconnected-(SW3-PadMP)_2: track 30.5 -> 0.00 mm
- net Net-(Q2-E): track 165.0 -> 160.7 mm
- net Net-(Q2-B): track 214.2 -> 210.4 mm
- net Net-(R5-Pad2): track 11.1 -> 13.8 mm
- net Net-(R7-Pad2): track 10.7 -> 13.3 mm
- net Net-(R8-Pad2): track 10.5 -> 11.5 mm
- net Net-(R9-Pad2): track 10.5 -> 11.4 mm
- net Net-(R6-Pad2): track 11.5 -> 12.1 mm
Other:
- outline, holes or cut-outs redrawn
